File: epc/base/camera_cape.sch (EAGLE design)
At the start: 17 parts, among them J1 MEC6, U1 MP2560

Commit message: backup
Parts:
- removed LED_10V: (no value), led:LEDSML0603
- added 10K: 15k, rcl:R-EU_R0603
- added C10, C12, C6, C9: 0.1u, rcl:C-EUC0603
- added C11, C3: 47u/10v, rcl:CPOL-EUCT3528
- added C4: 1u, rcl:C-EUC0603
- added L2, L3: 100nH, rcl:R-EU_R0603
- added LED_5V: (no value), led:LEDSML0603
- added R1: 33k, rcl:R-EU_R0603
- added U$1: MAX868, my_ic:MAX868
- R5, R7: value 15k -> 33k
- R6: value 680R -> 1k2
Connections:
- removed net +10V: C7.+, L1.2, R4.2, R7.1
- new net +5V: 10K.1, C3.+, C4.1, C7.+, L1.2, L2.2, R4.2
- new net -10V: C11.-, L3.1, R1.1
- new net N$10: U$1.!SHDN
- new net N$11: C9.1, U$1.C1+
- new net N$12: C6.1, L2.1, R7.2, U$1.IN
- new net N$13: C9.2, U$1.C1-
- new net N$14: C10.1, U$1.C2+
- new net N$15: C10.2, U$1.C2-
- new net N$16: C12.1, L3.2, U$1.OUT
- new net N$17: R1.2, R7.1, U$1.FB
- net GND: now also C11.+, C12.2, C3.-, C4.2, C6.2, LED_5V.C, U$1.GND, U$1.PGND; no longer LED_10V.C
- net N$9: now also 10K.2, LED_5V.A; no longer LED_10V.A, R7.2
Other:
- moved on the sheet: R7
